File: hw/Canta.kicad_pcb (KiCad board)
At the start: 2 copper layers, 85.6 x 54 mm, 51 parts, among them J1 USB_C_Receptacle_PowerOnly_6P, J101 Conn_01x01, J102 Conn_01x01, J103 Conn_01x01, J104 Conn_01x01, J105 Conn_01x01, J106 Conn_01x01, J107 Conn_01x01, J108 Conn_01x01, J109 Conn_01x01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

Commit message: Update component values with actual assembly
Parts:
- C1: value 100n -> 4.7u
- R101, R102, R103, R104, R105, R106, R107, R108, R109, R110, R111, R112: value 470k -> 1M
Changed lines of the file:
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@@
         (effects (font (size 1 1) (thickness 0.15)))
     )
-    (fp_text value "470k" (at 0 1.17 90) (layer "F.Fab")
+    (fp_text value "1M" (at 0 1.17 90) (layer "F.Fab")
         (effects (font (size 1 1) (thickness 0.15)))
     )
@@
         (effects (font (size 1 1) (thickness 0.15)))
     )
-    (fp_text value "470k" (at 0 1.17 90) (layer "F.Fab")
+    (fp_text value "1M" (at 0 1.17 90) (layer "F.Fab")
         (effects (font (size 1 1) (thickness 0.15)))
     )
@@
       )
     )
-    (fp_text value "470k" (at 0 1.17 90) (layer "F.Fab")
+    (fp_text value "1M" (at 0 1.17 90) (layer "F.Fab")
         (effects (font (size 1 1) (thickness 0.15)))
     )
@@
         (effects (font (size 1 1) (thickness 0.15)))
     )
-    (fp_text value "470k" (at 0 1.17 90) (layer "F.Fab")
+    (fp_text value "1M" (at 0 1.17 90) (layer "F.Fab")
         (effects (font (size 1 1) (thickness 0.15)))
     )
@@
         (effects (font (size 1 1) (thickness 0.15)))
     )
-    (fp_text value "470k" (at 0 1.17 90) (layer "F.Fab")
+    (fp_text value "1M" (at 0 1.17 90) (layer "F.Fab")
         (effects (font (size 1 1) (thickness 0.15)))
     )
@@
         (effects (font (size 1 1) (thickness 0.15)))
     )
-    (fp_text value "470k" (at 0 1.17 90) (layer "F.Fab")
+    (fp_text value "1M" (at 0 1.17 90) (layer "F.Fab")
         (effects (font (size 1 1) (thickness 0.15)))
     )
@@
       )
     )
-    (fp_text value "470k" (at 0 1.17 90) (layer "F.Fab")
+    (fp_text value "1M" (at 0 1.17 90) (layer "F.Fab")
         (effects (font (size 1 1) (thickness 0.15)))
     )
@@
         (effects (font (size 1 1) (thickness 0.15)))
     )
-    (fp_text value "470k" (at 0 1.17 90) (layer "F.Fab")
+    (fp_text value "1M" (at 0 1.17 90) (layer "F.Fab")
         (effects (font (size 1 1) (thickness 0.15)))
     )
@@
         (effects (font (size 1 1) (thickness 0.15)))
     )
-    (fp_text value "470k" (at 0 1.17 90) (layer "F.Fab")
+    (fp_text value "1M" (at 0 1.17 90) (layer "F.Fab")
         (effects (font (size 1 1) (thickness 0.15)))
     )
@@
         (effects (font (size 1 1) (thickness 0.15)))
     )
-    (fp_text value "470k" (at 0 1.17 90) (layer "F.Fab")
+    (fp_text value "1M" (at 0 1.17 90) (layer "F.Fab")
         (effects (font (size 1 1) (thickness 0.15)))
     )
@@
       )
     )
-    (fp_text value "100n" (at 0 1.16 90) (layer "F.Fab")
+    (fp_text value "4.7u" (at 0 1.16 90) (layer "F.Fab")
         (effects (font (size 1 1) (thickness 0.15)))
     )
@@
         (effects (font (size 1 1) (thickness 0.15)))
     )
-    (fp_text value "470k" (at 0 1.17 90) (layer "F.Fab")
+    (fp_text value "1M" (at 0 1.17 90) (layer "F.Fab")
         (effects (font (size 1 1) (thickness 0.15)))
     )
@@
         (effects (font (size 1 1) (thickness 0.15)))
     )
-    (fp_text value "470k" (at 0 1.17 90) (layer "F.Fab")
+    (fp_text value "1M" (at 0 1.17 90) (layer "F.Fab")
         (effects (font (size 1 1) (thickness 0.15)))
     )

Commit message: Revise hardware design
Parts:
- removed JP1, JP2: SolderJumper_2_Open, Canta_footprints:SolderJumper-2_Open
- removed R101, R102, R103, R104, R105, R106, R107, R108, R109, R110, R111, R112: 1M, Resistor_SMD:R_0402_1005Metric
- added C10: 1u, Capacitor_SMD:C_0402_1005Metric, F.Cu at (29.3, 21.4)
- added C11: 1u, Capacitor_SMD:C_0402_1005Metric, F.Cu at (34.4, 21.4)
- added RN1: 1M, Resistor_SMD:R_Array_Convex_4x0402, F.Cu at (34.1, 33.5)
- added RN2: 1M, Resistor_SMD:R_Array_Convex_4x0402, F.Cu at (37.9, 33.5)
- added RN3: 1M, Resistor_SMD:R_Array_Convex_4x0402, F.Cu at (42.4, 33.5)
- added U4: TLV70245_SOT23-5, Package_TO_SOT_SMD:SOT-23-5, F.Cu at (31.8, 21.9)
- moved J2 3.74 mm to (35.4, 25.5)
- moved R3 1.37 mm to (30.6, 24.1), turned to 0 degrees
- moved R1 0.59 mm to (28.6, 26.3)
- moved R2 0.56 mm to (28.6, 28.2)
- moved D1 0.56 mm to (28.8, 23.8), turned to 90 degrees
- turned LS1 to 0 degrees
Connections:
- C1 pad 1: +5V -> VDD
- C4 pad 1: +5V -> VDD
- C5 pad 1: +5V -> VDD
- C8 pad 1: +5V -> VDD
- D1 pad 2: +5V -> VDD
- J2 pad 2: SWCLK -> BTN_12
- J2 pad 3: SWDIO -> BTN_10
- U1 pad 6: +5V -> VDD
- U2 pad 5: +5V -> VDD
- U3 pad 6: +5V -> VDD
Routing:
- net VDD: track 0.00 -> 42.4 mm, vias 0 -> 4
- net +5V: track 55.1 -> 17.2 mm, vias 4 -> 0
- net GND: track 19.2 -> 23.7 mm, vias 46 -> 48
- net BTN_OUT: track 27.8 -> 32.3 mm, vias 13 -> 4
- net I2S_BCK: track 21.3 -> 16.9 mm
- net SWDIO: track 4.16 -> 0.00 mm, vias 2 -> 0
- net SWCLK: track 3.82 -> 0.00 mm, vias 2 -> 0
- net BTN_11: track 26.8 -> 30.0 mm
- net BTN_09: track 75.2 -> 76.8 mm
- net I2S_DATA: track 9.87 -> 8.55 mm
- net BTN_12: track 77.6 -> 76.4 mm
- net BTN_05: track 41.6 -> 42.8 mm
- net I2S_WS: track 10.0 -> 8.89 mm
- net BTN_08: track 66.6 -> 67.7 mm
- net Net-(U3-VO1): track 8.96 -> 10.00 mm
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Other:
- board text added: "24-SmSols"
- board text removed: "24-Awn"
- board text removed: "Canta-Cart"
- board text removed: "—"

Commit message: Revise pin assignment; submit for fab (Rev. 2)
Connections:
- U1 pad 11: BTN_OUT -> I2S_BCK
- U1 pad 12: BTN_11 -> BTN_OUT
- U1 pad 15: BTN_01 -> BTN_11
- U1 pad 16: BTN_02 -> BTN_01
- U1 pad 17: I2S_BCK -> BTN_02
Routing:
- net BTN_11: track 30.0 -> 18.2 mm
- net I2S_BCK: track 16.9 -> 12.2 mm, vias 2 -> 0
