File: hw/Canta.kicad_pcb (KiCad board)
At the start: 2 copper layers, 85.6 x 54 mm, 14 parts

Commit message: hw: Layout?
Parts:
- added C1: 100n, Capacitor_SMD:C_0402_1005Metric, F.Cu at (63.9, 56.2)
- added C2: 1u, Capacitor_SMD:C_0402_1005Metric, F.Cu at (63.9, 55.2)
- added C3: 1u, Capacitor_SMD:C_0402_1005Metric, F.Cu at (70.3, 51.9)
- added C4: 100n, Capacitor_SMD:C_0402_1005Metric, F.Cu at (68.9, 51.9)
- added C5: 100n, Capacitor_SMD:C_0402_1005Metric, F.Cu at (64.9, 51.9)
- added C6: 100n, Capacitor_SMD:C_0402_1005Metric, F.Cu at (60.2, 58.8)
- added C7: 1u, Capacitor_SMD:C_0402_1005Metric, F.Cu at (59.4, 53.2)
- added C8: 1u, Capacitor_SMD:C_0402_1005Metric, F.Cu at (63.4, 51.9)
- added D1: White, LED_SMD:LED_0603_1608Metric, F.Cu at (58.2, 48.8)
- added J2: USB_C_Receptacle_USB2.0_14P, Connector_USB:USB_C_Receptacle_HRO_TYPE-C-31-M-12, F.Cu at (53.0, 56.0)
- added R1: 4.7k, Resistor_SMD:R_0402_1005Metric, F.Cu at (63.9, 53.4)
- added R5: 5.1k, Resistor_SMD:R_0402_1005Metric, F.Cu at (59.2, 54.3)
- added R6: 5.1k, Resistor_SMD:R_0402_1005Metric, F.Cu at (59.3, 59.9)
- added RN1: 1M, Resistor_SMD:R_Array_Convex_4x0402, F.Cu at (65.0, 60.5)
- added RN2: 1M, Resistor_SMD:R_Array_Convex_4x0402, F.Cu at (68.3, 60.5)
- added RN3: 1M, Resistor_SMD:R_Array_Convex_4x0402, F.Cu at (71.8, 60.5)
- added SW1: SW_SPST, Canta_footprints:TestPoints_1x02_P1.50, F.Cu at (72.1, 56.8)
- added U1: CH591F, QFN-28-P0.4-EP2.7:QFN-28-1EP_4x4mm_P0.4mm_EP2.7x2.7mm, F.Cu at (67.5, 55.5)
- added U2: MAX98357A, Package_CSP:WLCSP-9_1.21x1.22mm_Layout3x3_P0.4mm, F.Cu at (66.4, 51.8)
- added U3: USBLC6-2SC6, Package_TO_SOT_SMD:SOT-23-6, F.Cu at (60.5, 56.6)
- added U4: ME6206A33XG, Package_TO_SOT_SMD:SOT-23, F.Cu at (61.0, 52.0)
- added Y1: 32MHz, Crystal:Crystal_SMD_2016-4Pin_2.0x1.6mm, F.Cu at (72.0, 54.5)
Connections:
- E01 pad 1: BTN_01 -> /CAP_01
- E02 pad 1: BTN_02 -> /CAP_02
- E03 pad 1: BTN_03 -> /CAP_03
- E04 pad 1: BTN_04 -> /CAP_04
- E05 pad 1: BTN_05 -> /CAP_05
- E06 pad 1: BTN_06 -> /CAP_06
- E07 pad 1: BTN_07 -> /CAP_07
- E08 pad 1: BTN_08 -> /CAP_08
- E09 pad 1: BTN_09 -> /CAP_09
- E10 pad 1: BTN_10 -> /CAP_10
- E11 pad 1: BTN_11 -> /CAP_11
- E12 pad 1: BTN_12 -> /CAP_12

Commit message: hw: Layout...?
Parts:
- moved D1 12.8 mm to (62.5, 60.9), turned to 180 degrees
- moved C7 2.95 mm to (62.0, 54.6), turned to 180 degrees
- moved R1 1.93 mm to (65.5, 54.5)
- moved C2 1.84 mm to (65.4, 56.2)
- moved C3 1.81 mm to (71.8, 52.9)
- moved U1 1.81 mm to (69.0, 56.5)
- moved C1 1.81 mm to (65.4, 57.1)
- moved C4 1.81 mm to (70.4, 52.9)
- moved U2 1.62 mm to (67.8, 52.5)
- moved Y1 1.62 mm to (73.4, 55.2)
- moved C5 1.54 mm to (66.4, 52.0), turned to -90 degrees
- moved SW1 1.53 mm to (73.5, 57.5)
- moved C8 1.17 mm to (64.5, 52.3)
- moved U4 1.17 mm to (62.1, 52.4)
- moved J2 1.08 mm to (54.0, 56.3)
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- renumbered R6 to R5, R5 to R6
Connections:
- R5 pad 1: Net-(J2-CC1) -> Net-(J2-CC2)
- R6 pad 1: Net-(J2-CC2) -> Net-(J2-CC1)

Commit message: hw: Some routing
Parts:
- removed SW1: SW_SPST, Canta_footprints:TestPoints_1x02_P1.50
- moved R1 5.14 mm to (63.6, 59.4)
- moved Y1 0.90 mm to (73.2, 56.1)
- moved D1 0.70 mm to (63.1, 60.6)
Connections:
- D1 pad 1: GND -> /BOOT_ACT
- R1 pad 1: /ACT_LED -> VDD
- U1 pad 17: /BOOT -> /BOOT_ACT
- U1 pad 28: /ACT_LED -> unconnected-(U1-PA12/SCS/PWM4/AIN2-Pad28)
Routing:
- net VBUS: track 0.00 -> 10.7 mm
- net GND: track 0.00 -> 9.59 mm, vias 0 -> 6
- net Net-(J2-D--PadA7): track 0.00 -> 5.24 mm, vias 0 -> 2
- net Net-(J2-D+-PadA6): track 0.00 -> 5.16 mm
- net /I2S_WS: track 0.00 -> 4.56 mm, vias 0 -> 2
- net Net-(U1-X32MO): track 0.00 -> 3.24 mm
- net Net-(J2-CC2): track 0.00 -> 3.03 mm, vias 0 -> 2
- net Net-(U1-VINTA): track 0.00 -> 2.94 mm
- net VDD: track 0.00 -> 2.74 mm
- net /I2S_DATA: track 0.00 -> 2.74 mm, vias 0 -> 2
- net Net-(U1-X32MI): track 0.00 -> 1.88 mm
- net Net-(J2-CC1): track 0.00 -> 1.88 mm
- net /I2S_BCK: track 0.00 -> 1.69 mm
- net /VDCID: track 0.00 -> 1.25 mm
- net /BOOT_ACT: track 0.00 -> 0.76 mm, vias 0 -> 1

Commit message: hw: ... > <
Parts:
- moved RN3 1.98 mm to (74.8, 60.2)
- moved RN2 0.99 mm to (70.3, 60.7)
- moved RN1 0.85 mm to (66.9, 60.7)
- moved C2 0.05 mm to (65.4, 56.1)
- moved C3 0.05 mm to (71.8, 52.8)
- moved C4 0.05 mm to (70.4, 52.8)
- moved C5 0.05 mm to (66.4, 51.9)
- moved U1 0.05 mm to (69.0, 56.4)
- moved Y1 0.05 mm to (73.2, 56.0)
Connections:
- U1 pad 10: unconnected-(U1-PB13/SCK0_/TXD1_/DCD_-Pad10) -> /CAP_04
- U1 pad 11: unconnected-(U1-PB12/SCS_/RXD1_/RI_-Pad11) -> /CAP_05
- U1 pad 14: unconnected-(U1-PB7/TXD0/PWM9-Pad14) -> /CAP_06
- U1 pad 15: unconnected-(U1-PB4/RXD0/PWM7-Pad15) -> /CAP_07
- U1 pad 16: unconnected-(U1-PB23/RST/TMR0_/PWM11-Pad16) -> /CAP_08
- U1 pad 23: unconnected-(U1-PA4/AIN0-Pad23) -> /CAP_09
- U1 pad 24: unconnected-(U1-PA5/AIN1-Pad24) -> /CAP_10
- U1 pad 25: unconnected-(U1-PA15/MISO/RXD0_/AIN5-Pad25) -> /CAP_12
- U1 pad 6: unconnected-(U1-PA8/RXD1-Pad6) -> /CAP_11
- U1 pad 7: unconnected-(U1-PA9/TMR0/TXD1-Pad7) -> /CAP_01
- U1 pad 8: unconnected-(U1-PB15/TCK/MISO_/DTR-Pad8) -> /CAP_02
- U1 pad 9: unconnected-(U1-PB14/TIO/MOSI_/PWM10/DSR-Pad9) -> /CAP_03
Routing:
- net /CAP_10: track 0.00 -> 15.6 mm
- net /CAP_09: track 0.00 -> 14.4 mm
- net VDD: track 2.74 -> 15.0 mm, vias 0 -> 2
- net /VDCID: track 1.25 -> 9.09 mm, vias 0 -> 2
- net GND: track 9.59 -> 17.0 mm, vias 6 -> 15
- net VBUS: track 10.7 -> 17.4 mm
- net /CAP_11: track 0.00 -> 5.63 mm
- net /CAP_01: track 0.00 -> 5.42 mm
- net /CAP_05: track 0.00 -> 5.31 mm
- net /CAP_OUT: track 0.00 -> 4.92 mm
- net /CAP_06: track 0.00 -> 4.69 mm
- net /CAP_07: track 0.00 -> 4.63 mm
- net /CAP_02: track 0.00 -> 4.59 mm
- net /CAP_04: track 0.00 -> 4.44 mm
- net /CAP_12: track 0.00 -> 4.36 mm
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
Commit message: hw: Almost done routing!
Parts:
- added LS1: Speaker, Canta_footprints:Speaker_Pads_P2.00, F.Cu at (92.8, 52.0)
Routing:
- net Net-(U2-OUTP): track 0.00 -> 28.4 mm
- net Net-(U2-OUTN): track 0.00 -> 25.5 mm
- net /CAP_OUT: track 4.92 -> 22.8 mm, vias 0 -> 4
- net /CAP_12: track 4.36 -> 18.5 mm
- net /BOOT_ACT: track 0.76 -> 10.8 mm, vias 1 -> 2
- net /USB_D-: track 1.01 -> 10.5 mm, vias 1 -> 2
- net /USB_D+: track 0.83 -> 9.63 mm, vias 1 -> 2
- net /CAP_09: track 14.4 -> 16.7 mm
- net /CAP_10: track 15.6 -> 17.8 mm
- net /CAP_08: track 4.13 -> 6.14 mm
- net GND: vias 15 -> 31

Commit message: hw: Submit for fab (Rev. 3)
Routing:
- net /CAP_10: track 17.8 -> 89.4 mm
- net /CAP_09: track 16.7 -> 82.7 mm
- net /CAP_08: track 6.14 -> 64.2 mm
- net /CAP_12: track 18.5 -> 76.0 mm
- net /CAP_07: track 4.63 -> 54.7 mm
- net /CAP_06: track 4.69 -> 46.8 mm
- net /CAP_05: track 5.31 -> 44.8 mm
- net /CAP_04: track 4.44 -> 40.7 mm
- net /CAP_01: track 5.42 -> 41.5 mm
- net /CAP_02: track 4.59 -> 38.1 mm
- net /CAP_03: track 4.10 -> 37.0 mm
- net /CAP_11: track 5.63 -> 22.6 mm
Other:
- board text added: "<25-"
- board text added: ">"
- board text added: "Rev. 3"
- board text added: "ayu.land/canta-cart"
- board text added: "夏至"
